File: PCB/Guardrail FC.kicad_pcb (KiCad board)
At the start: 2 copper layers, 0 parts

Commit message: PCB Done!
Parts:
- added C1: 100nF, Capacitor_SMD:C_0603_1608Metric_Pad1.08x0.95mm_HandSolder, F.Cu at (68.5, 57.5)
- added C10: 100nF, Capacitor_SMD:C_0603_1608Metric_Pad1.08x0.95mm_HandSolder, F.Cu at (60.2, 64.5)
- added C11: 100nF, Capacitor_SMD:C_0603_1608Metric_Pad1.08x0.95mm_HandSolder, F.Cu at (60.2, 60.2)
- added C12: 100nF, Capacitor_SMD:C_0603_1608Metric_Pad1.08x0.95mm_HandSolder, F.Cu at (65.6, 69.5)
- added C13: .1uF, Capacitor_SMD:C_0603_1608Metric_Pad1.08x0.95mm_HandSolder, F.Cu at (69.0, 90.8)
- added C14: 100nF, Capacitor_SMD:C_0603_1608Metric_Pad1.08x0.95mm_HandSolder, F.Cu at (69.7, 52.7)
- added C15: .1uF, Capacitor_SMD:C_0603_1608Metric_Pad1.08x0.95mm_HandSolder, F.Cu at (73.4, 88.2)
- added C16: 22uF, Capacitor_SMD:C_0603_1608Metric_Pad1.08x0.95mm_HandSolder, F.Cu at (73.4, 86.8)
- added C17: 20pF, Capacitor_SMD:C_0603_1608Metric_Pad1.08x0.95mm_HandSolder, F.Cu at (71.8, 83.8)
- added C18: 22uF, Capacitor_SMD:C_0603_1608Metric_Pad1.08x0.95mm_HandSolder, F.Cu at (71.8, 82.2)
- added C19: 22uF, Capacitor_SMD:C_0603_1608Metric_Pad1.08x0.95mm_HandSolder, F.Cu at (71.8, 80.8)
- added C2: 15pF, Capacitor_SMD:C_0603_1608Metric_Pad1.08x0.95mm_HandSolder, F.Cu at (63.4, 73.7)
- added C20: 1uF, Capacitor_SMD:C_0603_1608Metric_Pad1.08x0.95mm_HandSolder, F.Cu at (62.0, 81.5)
- added C21: 1uF, Capacitor_SMD:C_0603_1608Metric_Pad1.08x0.95mm_HandSolder, F.Cu at (69.2, 94.2)
- added C22: 100nF, Capacitor_SMD:C_0603_1608Metric_Pad1.08x0.95mm_HandSolder, F.Cu at (67.8, 94.2)
- added C23: 100nF, Capacitor_SMD:C_0603_1608Metric_Pad1.08x0.95mm_HandSolder, F.Cu at (52.5, 60.9)
- added C24: 100nF, Capacitor_SMD:C_0603_1608Metric_Pad1.08x0.95mm_HandSolder, F.Cu at (54.8, 65.8)
- added C25: 100nF, Capacitor_SMD:C_0603_1608Metric_Pad1.08x0.95mm_HandSolder, F.Cu at (55.5, 68.2)
- added C3: 100nF, Capacitor_SMD:C_0603_1608Metric_Pad1.08x0.95mm_HandSolder, F.Cu at (65.5, 57.5)
- added C4: 15pF, Capacitor_SMD:C_0603_1608Metric_Pad1.08x0.95mm_HandSolder, F.Cu at (69.1, 73.7)
- added C5: 1uF, Capacitor_SMD:C_0603_1608Metric_Pad1.08x0.95mm_HandSolder, F.Cu at (69.0, 68.2)
- added C6: 1uF, Capacitor_SMD:C_0603_1608Metric_Pad1.08x0.95mm_HandSolder, F.Cu at (72.8, 65.4)
- added C7: 100nF, Capacitor_SMD:C_0603_1608Metric_Pad1.08x0.95mm_HandSolder, F.Cu at (71.2, 65.4)
- added C8: 100nF, Capacitor_SMD:C_0603_1608Metric_Pad1.08x0.95mm_HandSolder, F.Cu at (71.8, 59.5)
- added C9: 100nF, Capacitor_SMD:C_0603_1608Metric_Pad1.08x0.95mm_HandSolder, F.Cu at (67.0, 57.5)
- added D1: LED_PWR, LED_SMD:LED_0603_1608Metric, F.Cu at (72.2, 94.2)
- added D2: LED_USR, LED_SMD:LED_0603_1608Metric, F.Cu at (72.0, 74.1)
- added D3: 1N5819WS, Diode_SMD:D_SOD-323, F.Cu at (59.8, 72.0)
- added D4: 1N5819WS, Diode_SMD:D_SOD-323, F.Cu at (76.4, 91.2)
- added G***: LOGO, LOGO, B.Cu at (75.0, 75.0)
- added H1: MountingHole, MountingHole:MountingHole_2.2mm_M2_Pad_Via, F.Cu at (75.0, 53.0)
- added H2: MountingHole, MountingHole:MountingHole_2.2mm_M2_Pad_Via, F.Cu at (88.5, 53.0)
- added H3: MountingHole, MountingHole:MountingHole_2.2mm_M2_Pad_Via, F.Cu at (88.5, 97.0)
- added J1: Conn_02x03_Odd_Even, imported_components:HDR-SMD_6P-P2.54-V, F.Cu at (83.2, 89.9)
- added J10: Conn_02x03_Odd_Even, imported_components:HDR-SMD_6P-P2.54-V, F.Cu at (93.7, 57.4)
- added J2: Conn_02x03_Odd_Even, imported_components:HDR-SMD_6P-P2.54-V, F.Cu at (83.2, 81.7)
- added J3: Conn_02x03_Odd_Even, imported_components:HDR-SMD_6P-P2.54-V, F.Cu at (83.2, 73.6)
- added J4: Conn_02x03_Odd_Even, imported_components:HDR-SMD_6P-P2.54-V, F.Cu at (83.2, 65.5)
- added J5: Conn_02x03_Odd_Even, imported_components:HDR-SMD_6P-P2.54-V, F.Cu at (83.2, 57.4)
- added J6: Conn_02x03_Odd_Even, imported_components:HDR-SMD_6P-P2.54-V, F.Cu at (93.7, 89.9)
- added J7: Conn_02x03_Odd_Even, imported_components:HDR-SMD_6P-P2.54-V, F.Cu at (93.7, 81.7)
- added J8: Conn_02x03_Odd_Even, imported_components:HDR-SMD_6P-P2.54-V, F.Cu at (93.7, 73.6)
- added J9: Conn_02x03_Odd_Even, imported_components:HDR-SMD_6P-P2.54-V, F.Cu at (93.7, 65.5)
- added JP1: PWR_Jumper, Jumper:SolderJumper-2_P1.3mm_Bridged2Bar_RoundedPad1.0x1.5mm, F.Cu at (74.2, 94.3)
- added L1: APH252012C1R5MP01, easyeda2kicad:IND-SMD_APH252012C3R3MP01, F.Cu at (70.6, 87.5)
- added NO GPS?: LOGO, LOGO, F.Cu at (57.2, 91.2)
- added R1: 1K, Resistor_SMD:R_0603_1608Metric_Pad0.98x0.95mm_HandSolder, F.Cu at (68.1, 71.0)
- added R10: 5K1, Resistor_SMD:R_0603_1608Metric_Pad0.98x0.95mm_HandSolder, F.Cu at (59.9, 77.0)
- added R11: 5K1, Resistor_SMD:R_0603_1608Metric_Pad0.98x0.95mm_HandSolder, F.Cu at (60.7, 73.8)
- added R2: 1K, Resistor_SMD:R_0603_1608Metric_Pad0.98x0.95mm_HandSolder, F.Cu at (57.4, 57.6)
- added R3: 1K, Resistor_SMD:R_0603_1608Metric_Pad0.98x0.95mm_HandSolder, F.Cu at (51.8, 57.8)
- added R4: 1k, Resistor_SMD:R_0603_1608Metric_Pad0.98x0.95mm_HandSolder, F.Cu at (70.8, 94.2)
- added R5: 1k, Resistor_SMD:R_0603_1608Metric_Pad0.98x0.95mm_HandSolder, F.Cu at (72.0, 70.8)
- added R6: 39k, Resistor_SMD:R_0603_1608Metric_Pad0.98x0.95mm_HandSolder, F.Cu at (70.0, 85.2)
- added R7: 12.5k, Resistor_SMD:R_0603_1608Metric_Pad0.98x0.95mm_HandSolder, F.Cu at (73.5, 85.2)
- added R8: 4.7k, Resistor_SMD:R_0603_1608Metric_Pad0.98x0.95mm_HandSolder, F.Cu at (56.0, 61.8)
- added R9: 4.7k, Resistor_SMD:R_0603_1608Metric_Pad0.98x0.95mm_HandSolder, F.Cu at (57.5, 61.8)
- added SW1: BTN_BOOT, imported_lcsc:SW-SMD_4P-L5.2-W5.2-P5.80-LS6.4, F.Cu at (60.9, 55.3)
- added SW2: BTN_RST, imported_lcsc:SW-SMD_4P-L5.2-W5.2-P5.80-LS6.4, F.Cu at (54.2, 54.4)
- added U1: RP2040, Package_DFN_QFN:QFN-56-1EP_7x7mm_P0.4mm_EP3.2x3.2mm, F.Cu at (66.2, 63.3)
- added U2: W25Q16JVUXIQ, Package_SON:Winbond_USON-8-1EP_3x2mm_P0.5mm_EP0.2x1.6mm, F.Cu at (66.2, 52.7)
- added U3: TMI3341, imported_lcsc:SOT-23-6_L2.9-W1.6-P0.95-LS2.8-BL, F.Cu at (71.8, 90.8)
- added U4: SPA06-003, imported_lcsc:LGA-8_L2.5-W2.0-P0.65_SPA06-003, F.Cu at (52.0, 63.4)
- added U5: ICM-42688P-HXY, imported_lcsc:LGA-14_L3.0-W2.5-P0.50-TL, F.Cu at (53.0, 68.0)
- added U6: SAM-M8Q-0, imported_lcsc:LCC-20_L15.5-W15.5-P1.90_SAM-M10Q-00B, F.Cu at (59.1, 91.2)
- added USB1: USB-TYPE-C-018, imported_lcsc:USB-C_SMD-TYPE-C-31-M-12, F.Cu at (55.0, 75.0)
- added Y1: X322512MOB4SI 12pF, Crystal:Crystal_SMD_3225-4Pin_3.2x2.5mm, F.Cu at (66.2, 73.7)
Routing:
- net +3.3V: track 0.00 -> 153.6 mm, vias 0 -> 5
- net +BATT: track 0.00 -> 130.2 mm, vias 0 -> 9
- net GND: track 0.00 -> 118.3 mm, vias 0 -> 61
- net GPIO7: track 0.00 -> 90.8 mm, vias 0 -> 2
- net GPIO20: track 0.00 -> 52.9 mm, vias 0 -> 4
- net GPIO19: track 0.00 -> 48.1 mm
- net GPIO22: track 0.00 -> 46.0 mm, vias 0 -> 4
- net GPIO0: track 0.00 -> 44.2 mm, vias 0 -> 2
- net GPIO1: track 0.00 -> 44.1 mm, vias 0 -> 2
- net GPIO21: track 0.00 -> 42.9 mm
- net GPIO2: track 0.00 -> 42.4 mm, vias 0 -> 2
- net GPIO9: track 0.00 -> 42.0 mm, vias 0 -> 4
- net GPIO8: track 0.00 -> 40.9 mm, vias 0 -> 2
- net RUN: track 0.00 -> 39.4 mm, vias 0 -> 2
- net GPIO23: track 0.00 -> 36.6 mm
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- added copper zone on B.Cu, net GND
- added copper zone on F.Cu, net GND
Other:
- board outline added: 50 x 50 mm
- board text added: "+"
- board text added: "BOOT"
- board text added: "Designed by: Logan Peterson"
- board text added: "GND"
- board text added: "Guardrail Flight Controller"
- board text added: "INPUT"
- board text added: "OUT"
- board text added: "RST"
- board text added: "SERVO"
- board text added: "SIG"
- board text added: "THROTTLE"

Commit message: README + Zine + Firmware Done!
Parts:
- added R12: 10K, Resistor_SMD:R_0603_1608Metric_Pad0.98x0.95mm_HandSolder, F.Cu at (87.5, 92.5)
- added R13: 20K, Resistor_SMD:R_0603_1608Metric_Pad0.98x0.95mm_HandSolder, F.Cu at (97.8, 92.5)
- added R14: 10K, Resistor_SMD:R_0603_1608Metric_Pad0.98x0.95mm_HandSolder, F.Cu at (78.8, 95.2)
- added R15: 20K, Resistor_SMD:R_0603_1608Metric_Pad0.98x0.95mm_HandSolder, F.Cu at (76.2, 96.2)
- added R16: 10K, Resistor_SMD:R_0603_1608Metric_Pad0.98x0.95mm_HandSolder, F.Cu at (87.7, 84.5)
- added R17: 20K, Resistor_SMD:R_0603_1608Metric_Pad0.98x0.95mm_HandSolder, F.Cu at (97.8, 84.4)
- added R18: 10K, Resistor_SMD:R_0603_1608Metric_Pad0.98x0.95mm_HandSolder, F.Cu at (77.0, 84.5)
- added R19: 20K, Resistor_SMD:R_0603_1608Metric_Pad0.98x0.95mm_HandSolder, F.Cu at (78.0, 81.8)
- added R20: 10K, Resistor_SMD:R_0603_1608Metric_Pad0.98x0.95mm_HandSolder, F.Cu at (87.7, 76.2)
- added R21: 20K, Resistor_SMD:R_0603_1608Metric_Pad0.98x0.95mm_HandSolder, F.Cu at (98.2, 76.3)
- added R22: 10K, Resistor_SMD:R_0603_1608Metric_Pad0.98x0.95mm_HandSolder, F.Cu at (78.5, 76.2)
- added R23: 20K, Resistor_SMD:R_0603_1608Metric_Pad0.98x0.95mm_HandSolder, F.Cu at (77.5, 73.8)
- added R24: 10K, Resistor_SMD:R_0603_1608Metric_Pad0.98x0.95mm_HandSolder, F.Cu at (87.5, 68.2)
- added R25: 20K, Resistor_SMD:R_0603_1608Metric_Pad0.98x0.95mm_HandSolder, F.Cu at (97.8, 68.1)
- added R26: 10K, Resistor_SMD:R_0603_1608Metric_Pad0.98x0.95mm_HandSolder, F.Cu at (78.8, 68.0)
- added R27: 20K, Resistor_SMD:R_0603_1608Metric_Pad0.98x0.95mm_HandSolder, F.Cu at (78.9, 65.5)
- added R28: 10K, Resistor_SMD:R_0603_1608Metric_Pad0.98x0.95mm_HandSolder, F.Cu at (93.0, 51.2)
- added R29: 20K, Resistor_SMD:R_0603_1608Metric_Pad0.98x0.95mm_HandSolder, F.Cu at (93.0, 52.8)
- added R30: 10K, Resistor_SMD:R_0603_1608Metric_Pad0.98x0.95mm_HandSolder, F.Cu at (83.3, 51.0)
- added R31: 20K, Resistor_SMD:R_0603_1608Metric_Pad0.98x0.95mm_HandSolder, F.Cu at (83.3, 52.5)
Connections:
- net GPIO17 renamed 3.3VGPIO17
- net GPIO18 renamed 3.3VGPIO18
- U1 pad 11: GPIO8 -> 3.3VGPIO8
- U1 pad 12: GPIO9 -> 3.3VGPIO9
- U1 pad 13: GPIO10 -> 3.3VGPIO10
- U1 pad 14: GPIO11 -> 3.3VGPIO11
- U1 pad 15: GPIO12 -> 3.3VGPIO12
- U1 pad 16: GPIO13 -> 3.3VGPIO13
- U1 pad 17: GPIO14 -> 3.3VGPIO14
- U1 pad 18: GPIO15 -> 3.3VGPIO15
- U1 pad 27: GPIO16 -> 3.3VGPIO16
- U1 pad 9: GPIO7 -> 3.3VGPIO7
Routing:
- net 3.3VGPIO7: track 0.00 -> 104.8 mm, vias 0 -> 3
- net GPIO7: track 90.8 -> 1.42 mm, vias 2 -> 0
- net 3.3VGPIO9: track 0.00 -> 54.8 mm, vias 0 -> 5
- net 3.3VGPIO11: track 0.00 -> 46.6 mm, vias 0 -> 3
- net 3.3VGPIO15: track 0.00 -> 45.6 mm, vias 0 -> 2
- net 3.3VGPIO13: track 0.00 -> 42.9 mm, vias 0 -> 3
- net 3.3VGPIO8: track 0.00 -> 41.9 mm, vias 0 -> 2
- net GPIO9: track 42.0 -> 1.82 mm, vias 4 -> 0
- net GPIO8: track 40.9 -> 1.66 mm, vias 2 -> 0
- net 3.3VGPIO10: track 0.00 -> 33.8 mm, vias 0 -> 2
- net GPIO11: track 33.5 -> 1.50 mm, vias 2 -> 0
- net 3.3VGPIO16: track 0.00 -> 30.8 mm, vias 0 -> 2
- net GPIO10: track 32.4 -> 3.17 mm, vias 2 -> 0
- net GPIO13: track 29.9 -> 1.31 mm, vias 2 -> 0
- net 3.3VGPIO12: track 0.00 -> 25.1 mm, vias 0 -> 2
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Other:
- board text added: "Logan Peterson"
- board text removed: "Designed by: Logan Peterson"
